Commit message: further updates

File: policypilot/description_files/urdf/29dof.urdf (robot description, URDF)
Before this commit: robot g1_29dof_rev_1_0, 55 links, 54 joints
Links:
- link head_link: geometry collision mesh filename=package://policypilot/description_files/meshes/head_link.STL; visual mesh filename=package://policypilot/description_files/meshes/head_link.STL
- link left_ankle_pitch_link: geometry collision mesh filename=package://policypilot/description_files/meshes/left_ankle_p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; visual mesh filename=package://policypilot/description_files/meshes/left_ankle_p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
- link left_ankle_roll_link: geometry collision sphere radius=0.005; collision sphere radius=0.005
- link left_elbow_link: geometry collision mesh filename=package://policypilot/description_files/meshes/left_elbow_l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; visual mesh filename=package://policypilot/description_files/meshes/left_elbow_l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
- link left_hip_pitch_link: geometry collision mesh filename=package://policypilot/description_files/meshes/left_hip_pit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; visual mesh filename=package://policypilot/description_files/meshes/left_hip_pit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
- link left_hip_roll_link: geometry collision mesh filename=package://policypilot/description_files/meshes/left_hip_rol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; visual mesh filename=package://policypilot/description_files/meshes/left_hip_rol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
- link left_hip_yaw_link: geometry collision mesh filename=package://policypilot/description_files/meshes/left_hip_yaw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; visual mesh filename=package://policypilot/description_files/meshes/left_hip_yaw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
- link left_knee_link: geometry collision mesh filename=package://policypilot/description_files/meshes/left_knee_li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; visual mesh filename=package://policypilot/description_files/meshes/left_knee_li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
- link left_rubber_hand: geometry visual mesh filename=package://policypilot/description_files/meshes/left_rubber_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
- link left_shoulder_pitch_link: geometry collision cylinder length=0.05 radius=0.03; visual mesh filename=package://policypilot/description_files/meshes/left_shoulde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
- link left_shoulder_roll_link: geometry collision cylinder length=0.03 radius=0.03; visual mesh filename=package://policypilot/description_files/meshes/left_shoulde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
- link left_shoulder_yaw_link: geometry collision mesh filename=package://policypilot/description_files/meshes/left_shoulde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; visual mesh filename=package://policypilot/description_files/meshes/left_shoulde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
- link left_wrist_pitch_link: geometry collision mesh filename=package://policypilot/description_files/meshes/left_wrist_p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; visual mesh filename=package://policypilot/description_files/meshes/left_wrist_p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
- link left_wrist_roll_link: geometry collision mesh filename=package://policypilot/description_files/meshes/left_wrist_r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; visual mesh filename=package://policypilot/description_files/meshes/left_wrist_r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
- link left_wrist_yaw_link: geometry collision mesh filename=package://policypilot/description_files/meshes/left_wrist_y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; visual mesh filename=package://policypilot/description_files/meshes/left_wrist_y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
- link logo_link: geometry collision mesh filename=package://policypilot/description_files/meshes/logo_link.STL; visual mesh filename=package://policypilot/description_files/meshes/logo_link.STL
- link pelvis: geometry visual mesh filename=package://policypilot/description_files/meshes/pelvis.STL
- link pelvis_contour_link: geometry collision mesh filename=package://policypilot/description_files/meshes/pelvis_conto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; visual mesh filename=package://policypilot/description_files/meshes/pelvis_conto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
- link right_ankle_pitch_link: geometry collision mesh filename=package://policypilot/description_files/meshes/right_ankle_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; visual mesh filename=package://policypilot/description_files/meshes/right_ankle_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
- link right_ankle_roll_link: geometry collision sphere radius=0.005; collision sphere radius=0.005
- link right_elbow_link: geometry collision mesh filename=package://policypilot/description_files/meshes/right_elbow_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; visual mesh filename=package://policypilot/description_files/meshes/right_elbow_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
- link right_hip_pitch_link: geometry collision mesh filename=package://policypilot/description_files/meshes/right_hip_pi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; visual mesh filename=package://policypilot/description_files/meshes/right_hip_pi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
- link right_hip_roll_link: geometry collision mesh filename=package://policypilot/description_files/meshes/right_hip_ro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; visual mesh filename=package://policypilot/description_files/meshes/right_hip_ro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
- link right_hip_yaw_link: geometry collision mesh filename=package://policypilot/description_files/meshes/right_hip_ya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; visual mesh filename=package://policypilot/description_files/meshes/right_hip_ya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
- link right_knee_link: geometry collision mesh filename=package://policypilot/description_files/meshes/right_knee_l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; visual mesh filename=package://policypilot/description_files/meshes/right_knee_l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
- link right_rubber_hand: geometry visual mesh filename=package://policypilot/description_files/meshes/right_rubber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
- link right_shoulder_pitch_link: geometry collision cylinder length=0.05 radius=0.03; visual mesh filename=package://policypilot/description_files/meshes/right_should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
- link right_shoulder_roll_link: geometry collision cylinder length=0.03 radius=0.03; visual mesh filename=package://policypilot/description_files/meshes/right_should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
- link right_shoulder_yaw_link: geometry collision mesh filename=package://policypilot/description_files/meshes/right_should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; visual mesh filename=package://policypilot/description_files/meshes/right_should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
- link right_wrist_pitch_link: geometry collision mesh filename=package://policypilot/description_files/meshes/right_wrist_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; visual mesh filename=package://policypilot/description_files/meshes/right_wrist_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
- link right_wrist_roll_link: geometry collision mesh filename=package://policypilot/description_files/meshes/right_wrist_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; visual mesh filename=package://policypilot/description_files/meshes/right_wrist_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
- link right_wrist_yaw_link: geometry collision mesh filename=package://policypilot/description_files/meshes/right_wrist_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; visual mesh filename=package://policypilot/description_files/meshes/right_wrist_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
- link torso_link: geometry collision mesh filename=package://policypilot/description_files/meshes/torso_link_r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; visual mesh filename=package://policypilot/description_files/meshes/torso_link_r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
- link waist_roll_link: geometry visual mesh filename=package://policypilot/description_files/meshes/waist_roll_l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
- link waist_yaw_link: geometry visual mesh filename=package://policypilot/description_files/meshes/waist_yaw_li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
